File: projects/kicad/docs.kicad_pcb (KiCad board)
At the start: 2 copper layers, 90 x 100 mm, 23 parts, among them SW1 SW_PUSH, SW2 SW_PUSH, SW3 SW_PUSH, SW4 SW_PUSH, SW5 SW_PUSH, SW6 SW_PUSH, SW7 RotaryEncoder_Switch, U1 Pico, U3 2.8_240x320_touch_sd_spi

Commit message: chocolate: Top plate および Bottom plate の作成
2/18 アップデート
Parts:
- added Ref**: Val**, kbd_Hole:m2_Screw_Hole_EdgeCuts, F.Cu at (128.0, 98.0)
- added Ref**: Val**, kbd_Hole:m2_Screw_Hole_EdgeCuts, F.Cu at (128.1, 252.4)
- added Ref**: Val**, kbd_hole:m2_Screw_Hole, F.Cu at (90.5, 130.5)
- added Ref**: Val**, kbd_Hole:m3_Screw_Hole_EdgeCuts, F.Cu at (137.0, 230.3)
- added Ref**: Val**, kbd_Hole:m3_Screw_Hole_EdgeCuts, F.Cu at (157.0, 126.0)
- added Ref**: Val**, kbd_Hole:m2_Screw_Hole_EdgeCuts, F.Cu at (127.6, 270.4)
- added Ref**: Val**, kbd_hole:m2_Screw_Hole, F.Cu at (175.5, 130.5)
- added Ref**: Val**, kbd_Hole:m2_Screw_Hole_EdgeCuts, F.Cu at (91.5, 98.2)
- added Ref**: Val**, kbd_Hole:m3_Screw_Hole_EdgeCuts, F.Cu at (153.0, 126.0)
- added Ref**: Val**, kbd_Hole:m2_Screw_Hole_EdgeCuts, F.Cu at (127.5, 116.0)
- added Ref**: Val**, kbd_Hole:m3_Screw_Hole_EdgeCuts, F.Cu at (98.0, 230.3)
- added Ref**: Val**, kbd_Hole:m3_Screw_Hole_EdgeCuts, F.Cu at (102.0, 230.3)
- added Ref**: Val**, kbd_Hole:m2_Screw_Hole_EdgeCuts, F.Cu at (91.6, 252.6)
- added Ref**: Val**, kbd_Hole:m3_Screw_Hole_EdgeCuts, F.Cu at (108.0, 126.0)
- added Ref**: Val**, kbd_Hole:m3_Screw_Hole_EdgeCuts, F.Cu at (112.0, 126.0)
- added Ref**: Val**, kbd_hole:m2_Screw_Hole, F.Cu at (175.5, 226.0)
- added Ref**: Val**, kbd_hole:m2_Screw_Hole, F.Cu at (90.5, 226.0)
- added Ref**: Val**, kbd_Hole:m3_Screw_Hole_EdgeCuts, F.Cu at (133.0, 230.3)
- added SW2: KEY_SWITCH, kbd_SW_Hole:SW_Hole_1u_JLC, F.Cu at (99.5, 262.0)
- added SW2: KEY_SWITCH, kbd_SW_Hole:SW_Hole_1u_JLC, F.Cu at (118.5, 243.0)
- added SW2: KEY_SWITCH, kbd_SW_Hole:SW_Hole_1u_JLC, F.Cu at (137.5, 262.0)
- added SW2: KEY_SWITCH, kbd_SW_Hole:SW_Hole_1u_JLC, F.Cu at (118.5, 262.0)
- added SW2: KEY_SWITCH, kbd_SW_Hole:SW_Hole_1u_JLC, F.Cu at (137.5, 243.0)
- added SW2: KEY_SWITCH, kbd_SW_Hole:SW_Hole_1u_JLC, F.Cu at (99.5, 243.0)
- moved Ref** 0.71 mm to (90.5, 25.5)
- moved Ref** 0.50 mm to (175.5, 121.0)
- moved SW1 0.13 mm to (99.3, 88.6)
- moved SW3 0.12 mm to (118.4, 88.6)
- moved SW5 0.10 mm to (137.5, 88.6)
Routing:
- net Cal1: track 155.6 -> 154.4 mm
Other:
- board size 90 x 100 mm -> 90 x 250 mm
